Commit message: Changed package finding syntax back to original

File: p3at_description/urdf/pioneer3at.urdf.xacro (robot description, xacro)
@@ -24,5 +24,5 @@
 			<origin xyz="0 0 0.177" rpy="0 0 0"/>
 			<geometry name="pioneer_geom">
-				<mesh filename="$(find p3at_description)/meshes/p3at_meshes/chassis.stl"/>
+				<mesh filename="package://p3at_description/meshes/p3at_meshes/chassis.stl"/>
 			</geometry>
 			<material name="ChassisRed">
@@ -33,5 +33,5 @@
 			<origin xyz="0 0 0.177" rpy="0 0 0"/>
 				<geometry>
-					<mesh filename="$(find p3at_description)/meshes/p3at_meshes/chassis.stl"/>
+					<mesh filename="package://p3at_description/meshes/p3at_meshes/chassis.stl"/>
 				</geometry>
 		</collision>
@@ -52,5 +52,5 @@
 			<origin xyz="0 0 0" rpy="0 0 0"/>
 			<geometry name="pioneer_geom">
-				<mesh filename="$(find p3at_description)/meshes/p3at_meshes/top.stl"/>
+				<mesh filename="package://p3at_description/meshes/p3at_meshes/top.stl"/>
 			</geometry>
 			<material name="TopBlack">
@@ -78,5 +78,5 @@
 			<origin xyz="0 0 0" rpy="0 0 0"/>
 			<geometry name="pioneer_geom">
-				<mesh filename="$(find p3at_description)/meshes/p3at_meshes/front_sonar.stl"/>
+				<mesh filename="package://p3at_description/meshes/p3at_meshes/front_sonar.stl"/>
 			</geometry>
 			<material name="SonarYellow">
@@ -103,5 +103,5 @@
 			<origin xyz="0 0 0" rpy="0 0 0"/>
 			<geometry name="pioneer_geom">
-				<mesh filename="$(find p3at_description)/meshes/p3at_meshes/back_sonar.stl"/>
+				<mesh filename="package://p3at_description/meshes/p3at_meshes/back_sonar.stl"/>
 			</geometry>
 			<material name="SonarYellow">
@@ -130,5 +130,5 @@
 		<origin xyz="0 0 0" rpy="0 0 0"/>
 		<geometry name="pioneer_geom">
-			<mesh filename="$(find p3at_description)/meshes/p3at_meshes/axle.stl"/>
+			<mesh filename="package://p3at_description/meshes/p3at_meshes/axle.stl"/>
 		</geometry>
 		<material name="AxleGrey">
@@ -155,5 +155,5 @@
 		<origin xyz="0 0 0" rpy="0 0 0"/>
 		<geometry name="pioneer_geom">
-			<mesh filename="$(find p3at_description)/meshes/p3at_meshes/${side}_hubcap.stl"/>
+			<mesh filename="package://p3at_description/meshes/p3at_meshes/${side}_hubcap.stl"/>
 		</geometry>
 		<material name="HubcapYellow">
@@ -180,5 +180,5 @@
 		<origin xyz="0 0 0" rpy="0 0 0"/>
 		<geometry name="pioneer_geom">
-			<mesh filename="$(find p3at_description)/meshes/p3at_meshes/wheel.stl"/>
+			<mesh filename="package://p3at_description/meshes/p3at_meshes/wheel.stl"/>
 		</geometry>
 		<material name="WheelBlack">
@@ -189,5 +189,5 @@
 		<origin xyz="0 0 0" rpy="${-3.1415927/2} 0 0"/>
 		<geometry>
-	    <!--mesh filename="$(find p3at_description)/meshes/p3at_meshes/wheel.stl"/-->
+	    <!--mesh filename="package://p3at_description/meshes/p3at_meshes/wheel.stl"/-->
 	    <cylinder radius="0.111" length="0.075"/>
 		</geometry>
@@ -217,5 +217,5 @@
 		<origin xyz="0 0 0" rpy="0 0 0"/>
 		<geometry name="pioneer_geom">
-			<mesh filename="$(find p3at_description)/meshes/p3at_meshes/axle.stl"/>
+			<mesh filename="package://p3at_description/meshes/p3at_meshes/axle.stl"/>
 		</geometry>
 		<material name="AxleGrey">
@@ -226,5 +226,5 @@
 		<origin xyz="0 0 0" rpy="0 0 0"/>
 		<geometry>
-			<mesh filename="$(find p3at_description)/meshes/p3at_meshes/axle.stl"/>
+			<mesh filename="package://p3at_description/meshes/p3at_meshes/axle.stl"/>
 		</geometry>
 	</collision>
@@ -248,5 +248,5 @@
 		<origin xyz="0 0 0" rpy="0 0 0"/>
 		<geometry name="pioneer_geom">
-			<mesh filename="$(find p3at_description)/meshes/p3at_meshes/${side}_hubcap.stl"/>
+			<mesh filename="package://p3at_description/meshes/p3at_meshes/${side}_hubcap.stl"/>
 		</geometry>
 		<material name="HubcapYellow"/>
@@ -255,5 +255,5 @@
 		<origin xyz="0 0 0" rpy="0 0 0"/>
 		<geometry>
-			<mesh filename="$(find p3at_description)/meshes/p3at_meshes/${side}_hubcap.stl"/>
+			<mesh filename="package://p3at_description/meshes/p3at_meshes/${side}_hubcap.stl"/>
 		</geometry>
 	</collision>
@@ -278,5 +278,5 @@
 		<origin xyz="0 0 0" rpy="0 0 0"/>
 		<geometry name="pioneer_geom">
-			<mesh filename="$(find p3at_description)/meshes/p3at_meshes/wheel.stl"/>
+			<mesh filename="package://p3at_description/meshes/p3at_meshes/wheel.stl"/>
 		</geometry>
 		<material name="WheelBlack"/>
@@ -285,5 +285,5 @@
 		<origin xyz="0 0 0" rpy="${-3.1415927/2} 0 0"/>
 		<geometry>
-	    <!--mesh filename="$(find p3at_description)/meshes/p3at_meshes/wheel.stl"/-->
+	    <!--mesh filename="package://p3at_description/meshes/p3at_meshes/wheel.stl"/-->
 	    <cylinder radius="0.111" length="0.075"/>
 		</geometry>

Commit message: created basic driver for ICM20948 IMU - requires manual install of ICM20948 python package

File: p3at_description/urdf/pioneer3at.urdf.xacro (robot description, xacro)
@@ -5,6 +5,10 @@
        xmlns:xacro="http://ros.org/wiki/xacro"
 name="pioneer3at">
+	<link name="base_link">
+	</link>
+	<gazebo reference="base_link">
+	</gazebo>
 <!-- Chassis -->
-	<link name="base_link">
+	<link name="chassis">
 		<!--  For pointers on inertial and gazebo-related parameters see
 		       * http://wiki.ros.org/urdf/Tutorials/Adding%20Physical%20and%20Collision%20Properties%20to%20a%20URDF%20Model
@@ -16,5 +20,5 @@
 		<inertial>
 			<mass value="21.5"/> <!-- P3AT 18.6kg plus three batteries @ 2.4kg each  minus four wheels @ 1.4 kg ea and top plate @ 0.1 kg-->
-			<origin xyz="-0.1 0 0.177"/>
+			<origin xyz="-0.1 0 0"/>
 			<inertia ixx="0.3338" ixy="0.0"     ixz="0.0"
 				              iyy="0.4783"  iyz="0.0"
@@ -22,5 +26,5 @@
 		</inertial>
 		<visual>
-			<origin xyz="0 0 0.177" rpy="0 0 0"/>
+			<origin xyz="0 0 0" rpy="0 0 0"/>
 			<geometry name="pioneer_geom">
 				<mesh filename="package://p3at_description/meshes/p3at_meshes/chassis.stl"/>
@@ -31,5 +35,5 @@
 		</visual>
 		<collision>
-			<origin xyz="0 0 0.177" rpy="0 0 0"/>
+			<origin xyz="0 0 0" rpy="0 0 0"/>
 				<geometry>
 					<mesh filename="package://p3at_description/meshes/p3at_meshes/chassis.stl"/>
@@ -37,7 +41,12 @@
 		</collision>
 	</link>
-	<gazebo reference="base_link">
+	<gazebo reference="chassis">
 		<material value="Gazebo/Red"/>
 	</gazebo>
+	<joint name="base_chassis_joint" type="fixed">
+		<origin xyz="0 0 0.177" rpy="0 0 0"/>
+		<parent link="base_link"/>
+		<child link="chassis"/>
+	</joint>
 <!-- Top -->
 	<link name="top_plate">
