Commit message: Added IMU link to xacro in separate file

File: p3at_description/urdf/p3at.urdf.xacro (robot description, xacro)
@@ -1,3 +1,10 @@
 <?xml version="1.0"?>
+<!--Original version from amr-ros-config package:
+https://github.com/MobileRobots/amr-ros-config/blob/master/description/urdf/pioneer3at.urdf.xacro
+Modifications:
+- Added include of p3at_customisation xacro file
+- Moved base_link inertial component to separate link (so KDL doesn't complain)
+- Added robot_namespace argument, used for Gazebo plugins
+-->
 <robot xmlns:sensor="http://playerstage.sourceforge.net/gazebo/xmlschema/#sensor"
        xmlns:controller="http://playerstage.sourceforge.net/gazebo/xmlschema/#controller"
@@ -5,26 +12,8 @@
        xmlns:xacro="http://ros.org/wiki/xacro"
 name="pioneer3at">
+	<xacro:arg name="robot_namespace" default="/" />
 	<link name="base_link">
-	</link>
-	<gazebo reference="base_link">
-	</gazebo>
-<!-- Chassis -->
-	<link name="chassis">
-		<!--  For pointers on inertial and gazebo-related parameters see
-		       * http://wiki.ros.org/urdf/Tutorials/Adding%20Physical%20and%20Collision%20Properties%20to%20a%20URDF%20Model
-                       * http://answers.gazebosim.org/question/4372/the-inertia-matrix-explained/
-		       * http://gazebosim.org/tutorials?tut=inertia&cat=build_robot, and
-                       * http://gazebosim.org/tutorials/?tut=ros_urdf
-                       * http://en.wikipedia.org/wiki/List_of_moment_of_inertia_tensors
-                -->
-		<inertial>
-			<mass value="21.5"/> <!-- P3AT 18.6kg plus three batteries @ 2.4kg each  minus four wheels @ 1.4 kg ea and top plate @ 0.1 kg-->
-			<origin xyz="-0.1 0 0"/>
-			<inertia ixx="0.3338" ixy="0.0"     ixz="0.0"
-				              iyy="0.4783"  iyz="0.0"
-				                            izz="0.3338"/>
-		</inertial>
 		<visual>
-			<origin xyz="0 0 0" rpy="0 0 0"/>
+			<origin xyz="0 0 0.177" rpy="0 0 0"/>
 			<geometry name="pioneer_geom">
 				<mesh filename="package://p3at_description/meshes/p3at_meshes/chassis.stl"/>
@@ -35,5 +24,5 @@
 		</visual>
 		<collision>
-			<origin xyz="0 0 0" rpy="0 0 0"/>
+			<origin xyz="0 0 0.177" rpy="0 0 0"/>
 				<geometry>
 					<mesh filename="package://p3at_description/meshes/p3at_meshes/chassis.stl"/>
@@ -41,12 +30,19 @@
 		</collision>
 	</link>
-	<gazebo reference="chassis">
+	<gazebo reference="base_link">
 		<material value="Gazebo/Red"/>
 	</gazebo>
-	<joint name="base_chassis_joint" type="fixed">
-		<origin xyz="0 0 0.177" rpy="0 0 0"/>
-		<parent link="base_link"/>
-		<child link="chassis"/>
-	</joint>
+	<link name="inertial_link">
+		<inertial>
+			<mass value="21.5"/> <!-- P3AT 18.6kg plus three batteries @ 2.4kg each  minus four wheels @ 1.4 kg ea and top plate @ 0.1 kg-->
+			<origin xyz="-0.1 0 0.177"/>
+			<inertia ixx="0.3338"	ixy="0.0" ixz="0.0" iyy="0.4783" iyz="0.0" izz="0.3338"/>
+		</inertial>
+	</link>
+  <joint name="inertial_joint" type="fixed">
+    <origin xyz="0 0 0" rpy="0 0 0" />
+    <parent link="base_link" />
+    <child link="inertial_link" />
+  </joint>
 <!-- Top -->
 	<link name="top_plate">
@@ -280,7 +276,5 @@
 			<mass value="1.2"/>
 			<origin xyz="0 0 0"/>
-			<inertia ixx="0.012411765597" ixy="0" ixz="0"
-                                                      iyy="0.015218160428" iyz="0"
-                                                                           izz="0.011763977943"/>
+			<inertia ixx="0.012411765597" ixy="0" ixz="0" iyy="0.015218160428" iyz="0" izz="0.011763977943"/>
       </inertial>
 	<visual>
@@ -345,5 +339,5 @@
   <plugin name="skid_steer_drive_controller" filename="libgazebo_ros_skid_steer_drive.so">
     <updateRate>100.0</updateRate>
-    <robotNamespace>sim_p3at</robotNamespace>
+    <robotNamespace>$(arg robot_namespace)</robotNamespace>
     <leftFrontJoint>p3at_front_left_wheel_joint</leftFrontJoint>
     <rightFrontJoint>p3at_front_right_wheel_joint</rightFrontJoint>
@@ -365,3 +359,4 @@
 <xacro:p3at_drive_side side="right" reflect="-1"/>
 <xacro:p3at_gazebo_ext/>
+<xacro:include filename="$(find p3at_description)/urdf/p3at_customisation.urdf.xacro"/>
 </robot>

Commit message: Changed mesh to dae type and added laser filter

File: p3at_description/urdf/p3at.urdf.xacro (robot description, xacro)
@@ -17,5 +17,5 @@
 			<origin xyz="0 0 0.177" rpy="0 0 0"/>
 			<geometry name="pioneer_geom">
-				<mesh filename="package://p3at_description/meshes/p3at_meshes/chassis.stl"/>
+				<mesh filename="package://p3at_description/models/p3at_models/chassis.dae"/>
 			</geometry>
 			<material name="ChassisRed">
@@ -57,5 +57,5 @@
 			<origin xyz="0 0 0" rpy="0 0 0"/>
 			<geometry name="pioneer_geom">
-				<mesh filename="package://p3at_description/meshes/p3at_meshes/top.stl"/>
+				<mesh filename="package://p3at_description/models//top.dae"/>
 			</geometry>
 			<material name="TopBlack">
@@ -83,5 +83,5 @@
 			<origin xyz="0 0 0" rpy="0 0 0"/>
 			<geometry name="pioneer_geom">
-				<mesh filename="package://p3at_description/meshes/p3at_meshes/front_sonar.stl"/>
+				<mesh filename="package://p3at_description/models/p3at_models/front_sonar.dae"/>
 			</geometry>
 			<material name="SonarYellow">
@@ -108,5 +108,5 @@
 			<origin xyz="0 0 0" rpy="0 0 0"/>
 			<geometry name="pioneer_geom">
-				<mesh filename="package://p3at_description/meshes/p3at_meshes/back_sonar.stl"/>
+				<mesh filename="package://p3at_description/models/p3at_models/back_sonar.dae"/>
 			</geometry>
 			<material name="SonarYellow">
@@ -135,5 +135,5 @@
 		<origin xyz="0 0 0" rpy="0 0 0"/>
 		<geometry name="pioneer_geom">
-			<mesh filename="package://p3at_description/meshes/p3at_meshes/axle.stl"/>
+			<mesh filename="package://p3at_description/models/p3at_models/axle.dae"/>
 		</geometry>
 		<material name="AxleGrey">
@@ -160,5 +160,5 @@
 		<origin xyz="0 0 0" rpy="0 0 0"/>
 		<geometry name="pioneer_geom">
-			<mesh filename="package://p3at_description/meshes/p3at_meshes/${side}_hubcap.stl"/>
+			<mesh filename="package://p3at_description/models/p3at_models/hubcap.dae"/>
 		</geometry>
 		<material name="HubcapYellow">
@@ -185,5 +185,5 @@
 		<origin xyz="0 0 0" rpy="0 0 0"/>
 		<geometry name="pioneer_geom">
-			<mesh filename="package://p3at_description/meshes/p3at_meshes/wheel.stl"/>
+			<mesh filename="package://p3at_description/models/p3at_models/wheel.dae"/>
 		</geometry>
 		<material name="WheelBlack">
@@ -194,5 +194,5 @@
 		<origin xyz="0 0 0" rpy="${-3.1415927/2} 0 0"/>
 		<geometry>
-	    <!--mesh filename="package://p3at_description/meshes/p3at_meshes/wheel.stl"/-->
+	    	<mesh filename="package://p3at_description/meshes/p3at_meshes/wheel.stl"/>
 	    <cylinder radius="0.111" length="0.075"/>
 		</geometry>
@@ -222,5 +222,5 @@
 		<origin xyz="0 0 0" rpy="0 0 0"/>
 		<geometry name="pioneer_geom">
-			<mesh filename="package://p3at_description/meshes/p3at_meshes/axle.stl"/>
+			<mesh filename="package://p3at_description/models/p3at_models/axle.dae"/>
 		</geometry>
 		<material name="AxleGrey">
@@ -253,5 +253,5 @@
 		<origin xyz="0 0 0" rpy="0 0 0"/>
 		<geometry name="pioneer_geom">
-			<mesh filename="package://p3at_description/meshes/p3at_meshes/${side}_hubcap.stl"/>
+			<mesh filename="package://p3at_description/models/p3at_models/hubcap.dae"/>
 		</geometry>
 		<material name="HubcapYellow"/>
@@ -281,5 +281,5 @@
 		<origin xyz="0 0 0" rpy="0 0 0"/>
 		<geometry name="pioneer_geom">
-			<mesh filename="package://p3at_description/meshes/p3at_meshes/wheel.stl"/>
+			<mesh filename="package://p3at_description/models/p3at_models/wheel.dae"/>
 		</geometry>
 		<material name="WheelBlack"/>
@@ -288,5 +288,5 @@
 		<origin xyz="0 0 0" rpy="${-3.1415927/2} 0 0"/>
 		<geometry>
-	    <!--mesh filename="package://p3at_description/meshes/p3at_meshes/wheel.stl"/-->
+	    	<mesh filename="package://p3at_description/meshes/p3at_meshes/wheel.stl"/>
 	    <cylinder radius="0.111" length="0.075"/>
 		</geometry>

Commit message: fixed xacro errors

File: p3at_description/urdf/p3at.urdf.xacro (robot description, xacro)
@@ -17,5 +17,5 @@
 			<origin xyz="0 0 0.177" rpy="0 0 0"/>
 			<geometry name="pioneer_geom">
-				<mesh filename="package://p3at_description/models/p3at_models/chassis.dae"/>
+				<mesh filename="package://p3at_description/meshes/p3at_meshes/chassis.stl"/>
 			</geometry>
 			<material name="ChassisRed">
@@ -57,5 +57,5 @@
 			<origin xyz="0 0 0" rpy="0 0 0"/>
 			<geometry name="pioneer_geom">
-				<mesh filename="package://p3at_description/models//top.dae"/>
+				<mesh filename="package://p3at_description/meshes/p3at_meshes/top.stl"/>
 			</geometry>
 			<material name="TopBlack">
@@ -83,5 +83,5 @@
 			<origin xyz="0 0 0" rpy="0 0 0"/>
 			<geometry name="pioneer_geom">
-				<mesh filename="package://p3at_description/models/p3at_models/front_sonar.dae"/>
+				<mesh filename="package://p3at_description/meshes/p3at_meshes/front_sonar.stl"/>
 			</geometry>
 			<material name="SonarYellow">
@@ -108,5 +108,5 @@
 			<origin xyz="0 0 0" rpy="0 0 0"/>
 			<geometry name="pioneer_geom">
-				<mesh filename="package://p3at_description/models/p3at_models/back_sonar.dae"/>
+				<mesh filename="package://p3at_description/meshes/p3at_meshes/back_sonar.stl"/>
 			</geometry>
 			<material name="SonarYellow">
@@ -135,5 +135,5 @@
 		<origin xyz="0 0 0" rpy="0 0 0"/>
 		<geometry name="pioneer_geom">
-			<mesh filename="package://p3at_description/models/p3at_models/axle.dae"/>
+			<mesh filename="package://p3at_description/meshes/p3at_meshes/axle.stl"/>
 		</geometry>
 		<material name="AxleGrey">
@@ -160,5 +160,5 @@
 		<origin xyz="0 0 0" rpy="0 0 0"/>
 		<geometry name="pioneer_geom">
-			<mesh filename="package://p3at_description/models/p3at_models/hubcap.dae"/>
+			<mesh filename="package://p3at_description/meshes/p3at_meshes/${side}_hubcap.stl"/>
 		</geometry>
 		<material name="HubcapYellow">
@@ -185,5 +185,5 @@
 		<origin xyz="0 0 0" rpy="0 0 0"/>
 		<geometry name="pioneer_geom">
-			<mesh filename="package://p3at_description/models/p3at_models/wheel.dae"/>
+			<mesh filename="package://p3at_description/meshes/p3at_meshes/wheel.stl"/>
 		</geometry>
 		<material name="WheelBlack">
@@ -194,5 +194,5 @@
 		<origin xyz="0 0 0" rpy="${-3.1415927/2} 0 0"/>
 		<geometry>
-	    	<mesh filename="package://p3at_description/meshes/p3at_meshes/wheel.stl"/>
+	    <!--mesh filename="package://p3at_description/meshes/p3at_meshes/wheel.stl"/-->
 	    <cylinder radius="0.111" length="0.075"/>
 		</geometry>
@@ -222,5 +222,5 @@
 		<origin xyz="0 0 0" rpy="0 0 0"/>
 		<geometry name="pioneer_geom">
-			<mesh filename="package://p3at_description/models/p3at_models/axle.dae"/>
+			<mesh filename="package://p3at_description/meshes/p3at_meshes/axle.stl"/>
 		</geometry>
 		<material name="AxleGrey">
@@ -253,5 +253,5 @@
 		<origin xyz="0 0 0" rpy="0 0 0"/>
 		<geometry name="pioneer_geom">
-			<mesh filename="package://p3at_description/models/p3at_models/hubcap.dae"/>
+			<mesh filename="package://p3at_description/meshes/p3at_meshes/${side}_hubcap.stl"/>
 		</geometry>
 		<material name="HubcapYellow"/>
@@ -281,5 +281,5 @@
 		<origin xyz="0 0 0" rpy="0 0 0"/>
 		<geometry name="pioneer_geom">
-			<mesh filename="package://p3at_description/models/p3at_models/wheel.dae"/>
+			<mesh filename="package://p3at_description/meshes/p3at_meshes/wheel.stl"/>
 		</geometry>
 		<material name="WheelBlack"/>
@@ -288,5 +288,5 @@
 		<origin xyz="0 0 0" rpy="${-3.1415927/2} 0 0"/>
 		<geometry>
-	    	<mesh filename="package://p3at_description/meshes/p3at_meshes/wheel.stl"/>
+	    <!--mesh filename="package://p3at_description/meshes/p3at_meshes/wheel.stl"/-->
 	    <cylinder radius="0.111" length="0.075"/>
 		</geometry>

File: p3at_description/urdf/p3at.xacro (robot description, xacro)
@@ -1,5 +1,6 @@
 <?xml version="1.0"?>
-<robot xmlns:xacro="http://www.ros.org/wiki/xacro" name="p3at_tutorial">
+<robot xmlns:xacro="http://ros.org/wiki/xacro" name="p3at">
 <xacro:property name="M_PI" value="3.1415926535897931" />
+<xacro:arg name="robot_namespace" default="/" />
 <xacro:include filename="$(find p3at_description)/urdf/pioneer3at_body.xacro"/>
 <xacro:p3at_front suffix="left" reflect="1"/>

File: p3at_description/urdf/p3at_test.urdf (robot description, URDF)
Before this commit: robot p3at_tutorial, 17 links, 16 joints
Links:
- added link imu
Joints:
- added joint imu_joint: type fixed, parent top_plate, child imu, origin xyz=-0.1 0 -0.01 rpy=0 0 -1.571
- joint chassis_top_joint: origin xyz=0.043 0 0.254 rpy=0 0 0 -> xyz=0.003 0 0.254 rpy=0 0 0
- joint rplidar_joint: origin xyz=0 0 0 rpy=0 0 0 -> xyz=0.21 0 -0.05 rpy=0 0 -1.571

File: p3at_description/urdf/pioneer3at_body.xacro (robot description, xacro)
@@ -46,5 +46,5 @@
 		</inertial>
 		<visual>
-			<origin xyz="0 0 0" rpy="0 0 0"/>
+			<origin xyz="0.04 0 0" rpy="0 0 0"/>
 			<geometry name="pioneer_geom">
 				<mesh filename="package://p3at_description/meshes/p3at_meshes/top.dae"/>
@@ -65,5 +65,5 @@
 	</gazebo>
 	<joint name="chassis_top_joint" type="fixed">
-		<origin xyz="0.043 0 0.254" rpy="0 0 0"/>
+		<origin xyz="0.003 0 0.254" rpy="0 0 0"/>
 		<parent link="base_link"/>
 		<child link="top_plate"/>
@@ -286,5 +286,5 @@
 </xacro:macro>
 <xacro:macro name="p3at_gazebo_ext">
-	<gazebo>
+	<!--gazebo>
 		<plugin name="joint_state_publisher" filename="libgazebo_ros_joint_state_publisher.so">
 		<robotNamespace></robotNamespace>
@@ -297,5 +297,5 @@
 	<plugin name="skid_steer_drive_controller" filename="libgazebo_ros_skid_steer_drive.so">
 		<updateRate>50.0</updateRate>
-		<!-- <robotNamespace>/</robotNamespace> -->
+		<robotNamespace>/</robotNamespace>
 		<leftFrontJoint>p3at_front_left_wheel_joint</leftFrontJoint>
 		<rightFrontJoint>p3at_front_right_wheel_joint</rightFrontJoint>
@@ -334,5 +334,5 @@
 			<headingGaussianNoise>0.05</headingGaussianNoise>
 		</plugin>
-	</gazebo>
+	</gazebo-->
 </xacro:macro>
 </robot>
